File: spindle-controller/Spindle_Controller.kicad_sch (KiCad schematic)
At the start: 24 parts, among them J1 Conn_01x19, J10 Conn_01x03, J11 Conn_01x02, J12 Conn_01x04, J13 Conn_01x02, J14 Conn_01x04, J15 GX12-7, J19 GX12-4, J2 Conn_01x19, J20 DIN-3, J21 DIN-3, J26 GX12-2, J3 Conn_01x14, J4 Jack-DC, J5 USB_C_Receptacle_USB2.0_16P, J6 Conn_01x04, J7 Conn_01x04, J8 Conn_01x04, J9 Conn_01x05, K2 JQC-3FF-005-1Z, K3 JQC-3FF-005-1Z, K4 JQC-3FF-005-1Z, K5 JQC-3FF-005-1Z, SW1 DPDT Toggle Switch

Commit message: test
Parts:
- removed J15: GX12-7, symbol GX12_Connectors:GX12-7
- added J18: GX16-8, symbol GX_Connectors:GX16-8
Connections:
- net LED_PLUS is gone; now on net VFD_24V: J19.1
- net VFD_24V: now also J18.5
- net VFD_COM: now also J18.6
- net VFD_DI1: now also J18.7
- net VFD_FM1: now also J18.2
- net VFD_GND: now also J18.4
- net VFD_RUN_SENSE: now also J18.1
- net VFD_VF1: now also J18.3
- no-connect marks 22 -> 23
Other:
- added sheet Original Spindle Controller (OriginalSpindleController.kicad_sch)
- note added: "LED Control"
- note added: "Spindle Control"
- note added: "Spindle Off"
- note added: "Spindle On"

Commit message: added the FOB circuit
Parts:
- added J27: GX12-2, symbol Connector:LEMO2
Connections:
- net at K2.11: now also J27.1
- net at K2.14: now also J27.2
- no-connect marks 23 -> 21
Other:
- note added: "Connected to FOB "Input""
- note added: "Connected to FOB GND"
- note added: "FOB "ON Signal""
- note removed: "Unused"
Changed lines of the file:
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@@
 		)
 	)
+	(text "Connected to FOB GND"
+		(exclude_from_sim no)
+		(at 194.31 193.294 0)
+		(effects
+			(font
+				(size 1.27 1.27)
+			)
+		)
+	)
 	(text "TechoCNC Controller\nCable"
 		(exclude_from_sim no)
@@
 		)
 	)
-	(text "Unused"
-		(exclude_from_sim no)
-		(at 139.954 85.852 0)
-		(effects
-			(font
-				(size 1.27 1.27)
-			)
-		)
-	)
 	(text "Green Wire"
 		(exclude_from_sim no)
@@
 		)
 	)
+	(text "FOB \"ON Signal\""
+		(exclude_from_sim no)
+		(at 168.402 181.864 0)
+		(effects
+			(font
+				(size 1.27 1.27)
+			)
+		)
+	)
 	(text "Orange Wire"
 		(exclude_from_sim no)
@@
 		)
 	)
+	(text "Relay #3"
+		(exclude_from_sim no)
+		(at 116.332 86.106 0)
+		(effects
+			(font
+				(size 1.27 1.27)
+			)
+		)
+	)
 	(text "Yellow Wire"
 		(exclude_from_sim no)
@@
 		)
 	)
+	(text "Connected to FOB \"Input\""
+		(exclude_from_sim no)
+		(at 194.564 164.846 0)
+		(effects
+			(font
+				(size 1.27 1.27)
+			)
+		)
+	)
 	(text "Green Wire"
 		(exclude_from_sim no)
@@
 	(text "Relay #4"
 		(exclude_from_sim no)
-		(at 115.824 88.646 0)
+		(at 203.454 183.896 0)
 		(effects
 			(font
@@
 	)
 	(no_connect
-		(at 128.27 77.47)
-	)
-	(no_connect
 		(at 246.38 124.46)
 	)
@@
 	)
 	(no_connect
-		(at 125.73 92.71)
-	)
-	(no_connect
 		(at 241.3 31.75)
 	)
@@
 	)
 	(no_connect
-		(at 123.19 77.47)
+		(at 210.82 172.72)
 	)
 	(no_connect
@@
 	(wire
 		(pts
+			(xy 284.48 77.0374) (xy 284.48 160.02)
+		)
+		(stroke
+			(width 0)
+			(type default)
+		)
+	)
+	(wire
+		(pts
 			(xy 161.29 41.91) (xy 161.29 58.42)
 		)
@@
 	(wire
 		(pts
+			(xy 215.9 167.64) (xy 215.9 172.72)
+		)
+		(stroke
+			(width 0)
+			(type default)
+		)
+	)
+	(wire
+		(pts
 			(xy 194.056 61.6367) (xy 176.53 61.6367)
 		)
@@
 	(wire
 		(pts
+			(xy 227.076 77.0374) (xy 284.48 77.0374)
+		)
+		(stroke
+			(width 0)
+			(type default)
+		)
+	)
+	(wire
+		(pts
 			(xy 186.5071 106.68) (xy 257.81 106.68)
 		)
@@
 	(wire
 		(pts
+			(xy 176.53 190.5) (xy 213.36 190.5)
+		)
+		(stroke
+			(width 0)
+			(type default)
+		)
+	)
+	(wire
+		(pts
 			(xy 58.42 40.64) (xy 72.39 40.64)
 		)
@@
 		)
 	)
+	(wire
+		(pts
+			(xy 176.53 167.64) (xy 215.9 167.64)
+		)
+		(stroke
+			(width 0)
+			(type default)
+		)
+	)
 	(polyline
 		(pts
@@
 	(wire
 		(pts
+			(xy 213.36 190.5) (xy 213.36 187.96)
+		)
+		(stroke
+			(width 0)
+			(type default)
+		)
+	)
+	(wire
+		(pts
 			(xy 139.7 148.59) (xy 173.99 148.59)
 		)
@@
 	(wire
 		(pts
+			(xy 176.53 182.88) (xy 176.53 190.5)
+		)
+		(stroke
+			(width 0)
+			(type default)
+		)
+	)
+	(wire
+		(pts
 			(xy 39.37 109.22) (xy 266.7 109.22)
 		)
@@
 	(wire
 		(pts
+			(xy 176.53 180.34) (xy 176.53 167.64)
+		)
+		(stroke
+			(width 0)
+			(type default)
+		)
+	)
+	(wire
+		(pts
 			(xy 254 23.591) (xy 254 31.75)
 		)
@@
 	)
 	(symbol
+		(lib_id "Connector:LEMO2")
+		(at 184.15 180.34 0)
+		(mirror x)
+		(unit 1)
+		(body_style 1)
+		(exclude_from_sim no)
+		(in_bom yes)
+		(on_board yes)
+		(in_pos_files yes)
+		(dnp no)
+		(property "Reference" "J27"
+			(at 188.976 182.8801 0)
+			(hide yes)
+			(show_name no)
+			(do_not_autoplace no)
+			(effects
+				(font
+					(size 1.27 1.27)
+				)
+				(justify left)
+			)
+		)
+		(property "Value" "GX12-2"
+			(at 183.5785 175.26 0)
+			(show_name no)
+			(do_not_autoplace no)
+			(effects
+				(font
+					(size 1.27 1.27)
+				)
+			)
+		)
+		(property "Footprint" ""
+			(at 184.15 181.61 0)
+			(hide yes)
+			(show_name no)
+			(do_not_autoplace no)
+			(effects
+				(font
+					(size 1.27 1.27)
+				)
+			)
+		)
+		(property "Datasheet" ""
+			(at 184.15 181.61 0)
+			(hide yes)
+			(show_name no)
+			(do_not_autoplace no)
+			(effects
+				(font
+					(size 1.27 1.27)
+				)
+			)
+		)
+		(property "Description" "2-pin LEMO connector"
+			(at 184.15 180.34 0)
+			(hide yes)
+			(show_name no)
+			(do_not_autoplace no)
+			(effects
+				(font
+					(size 1.27 1.27)
+				)
+			)
+		)
+		(pin "2"
+		)
+		(pin "1"
+		)
+		(instances
+			(project "Spindle_Controller"
+				(path "/10c7a81d-d8e0-4023-94dc-af5199d847de"
+					(reference "J27")
+					(unit 1)
+				)
+			)
+		)
+	)
+	(symbol
 		(lib_name "Conn_01x04_1")
 		(lib_id "Connector_Generic:Conn_01x04")
@@
 		(lib_name "JQC-3FF-005-1Z_1")
 		(lib_id "Relay:JQC-3FF-005-1Z")
-		(at 120.65 85.09 0)
+		(at 208.28 180.34 0)
 		(unit 1)
 		(body_style 1)
@@
 		(fields_autoplaced yes)
 		(property "Reference" "K2"
-			(at 132.08 83.8199 0)
+			(at 219.71 179.0699 0)
 			(hide yes)
 			(show_name no)
@@
 		)
 		(property "Value" "JQC-3FF-005-1Z"
-			(at 132.08 86.3599 0)
+			(at 219.71 181.6099 0)
 			(hide yes)
 			(show_name no)
@@
 		)
 		(property "Footprint" "Relay_THT:Relay_SPDT_Hongfa_JQC-3FF_0XX-1Z"
-			(at 132.08 86.36 0)
+			(at 219.71 181.61 0)
 			(hide yes)
 			(show_name no)
@@
 		)
 		(property "Datasheet" "https://www.digikey.com/htmldatasheets/production/2071105/0/0/1/JQC-3FF.pdf"
-			(at 120.65 85.09 0)
+			(at 208.28 180.34 0)
 			(hide yes)
 			(show_name no)
@@
 		)
 		(property "Description" "Subminiature High Power SPDT Relay, 5V Coil nom. 0.36W, 10A switching current, max 10A@277VAC/28VDC"
-			(at 120.65 85.09 0)
+			(at 208.28 180.34 0)
 			(hide yes)
 			(show_name no)
