File: spindle-controller/VFDEnclosure.kicad_sch (KiCad schematic)
At the start: 3 parts, among them J16 Conn_01x11, J23 Conn_01x03, J24 GX12-7

Commit message: test
Parts:
- removed J24: GX12-7, symbol GX12_Connectors:GX12-7
- added J17: GX16-8, symbol GX_Connectors:GX16-8
Connections:
- net VFD_24V: now also J17.5
- net VFD_COM: now also J17.6
- net VFD_DI1: now also J17.7
- net VFD_FM1: now also J17.2
- net VFD_GND: now also J23.1 (TA), J17.4; no longer J23.2 (TB)
- net VFD_RUN_SENSE: now also J23.2 (TB), J17.1; no longer J23.1 (TA)
- net VFD_VF1: now also J17.3
- net VFD_TC: now reaches J23.3 (TC)
- net VFD_TC: now also J17.8
- no-connect marks 1 -> 5
Other:
- note added: "Black wire"
- note added: "Blue wire"
- note added: "Brown wire"
- note added: "Green wire"
- note added: "Orange wire"
- note added: "Red wire"
- note added: "White wire"
- note added: "Yellow wire"

Commit message: wiring changes
Connections:
- net VFD_24V: now also J16.10 (OP)
- net VFD_COM: now also J16.9 (DI4)
- no-connect marks 5 -> 3
Changed lines of the file:
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@@
+	)
+	(junction
+		(at 80.01 50.8)
+		(diameter 0)
+		(color 0 0 0 0)
 	)
 	(junction
@@
 		(color 0 0 0 0)
 	)
-	(no_connect
-		(at 90.17 49.53)
+	(junction
+		(at 95.25 49.53)
+		(diameter 0)
+		(color 0 0 0 0)
 	)
 	(no_connect
@@
 	)
 	(no_connect
-		(at 92.71 49.53)
-	)
-	(no_connect
 		(at 85.09 49.53)
 	)
@@
 	(wire
 		(pts
+			(xy 92.71 49.53) (xy 95.25 49.53)
+		)
+		(stroke
+			(width 0)
+			(type default)
+		)
+	)
+	(wire
+		(pts
 			(xy 44.45 102.87) (xy 44.45 107.95)
 		)
@@
 	(wire
 		(pts
-			(xy 80.01 49.53) (xy 80.01 58.42)
+			(xy 80.01 49.53) (xy 80.01 50.8)
 		)
 		(stroke
@@
 	(wire
 		(pts
+			(xy 90.17 49.53) (xy 90.17 50.8)
+		)
+		(stroke
+			(width 0)
+			(type default)
+		)
+	)
+	(wire
+		(pts
 			(xy 120.65 35.56) (xy 29.21 35.56)
 		)
@@
 	(wire
 		(pts
+			(xy 80.01 50.8) (xy 80.01 58.42)
+		)
+		(stroke
+			(width 0)
+			(type default)
+		)
+	)
+	(wire
+		(pts
 			(xy 87.63 54.61) (xy 74.93 54.61)
 		)
@@
 		)
 		(stroke
+			(width 0)
+			(type default)
+		)
+	)
+	(wire
+		(pts
+			(xy 90.17 50.8) (xy 80.01 50.8)
+		)
+		(stroke
